File: mmc5983ma/mmc5983ma.kicad_sch (KiCad schematic)
At the start: 7 parts, among them J1 Conn_01x07, U1 MMC5983MA

Commit message: Slight modification to mmc and add ICP-20100
Changed lines of the file:
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@@
     (stroke (width 0) (type default) (color 0 0 0 0))
   )
-  (wire (pts (xy 187.325 78.74) (xy 196.215 78.74))
+  (wire (pts (xy 185.42 78.74) (xy 196.215 78.74))
     (stroke (width 0) (type default) (color 0 0 0 0))
   )
@@
     (effects (font (size 1.27 1.27)) (justify left bottom))
   )
-  (symbol (lib_id "power:+3V3") (at 187.325 78.74 90) (unit 1)
+  (symbol (lib_id "power:+3V3") (at 185.42 78.74 0) (unit 1)
     (in_bom yes) (on_board yes) (fields_autoplaced)
-    (property "Reference" "#PWR011" (id 0) (at 191.135 78.74 0)
+    (property "Reference" "#PWR011" (id 0) (at 185.42 82.55 0)
       (effects (font (size 1.27 1.27)) hide)
     )
-    (property "Value" "+3V3" (id 1) (at 183.515 78.7399 90)
-      (effects (font (size 1.27 1.27)) (justify left))
-    )
-    (property "Footprint" "" (id 2) (at 187.325 78.74 0)
+    (property "Value" "+3V3" (id 1) (at 185.42 73.66 0))
+    (property "Footprint" "" (id 2) (at 185.42 78.74 0)
       (effects (font (size 1.27 1.27)) hide)
     )
-    (property "Datasheet" "" (id 3) (at 187.325 78.74 0)
+    (property "Datasheet" "" (id 3) (at 185.42 78.74 0)
       (effects (font (size 1.27 1.27)) hide)
     )
