File: icp-20100/icp-20100.kicad_pcb (KiCad board)
At the start: 2 copper layers, 14.5 x 20.5 mm, 5 parts, among them J1 Conn_01x07, U1 ICP20100

Commit message: Slight modifications to boards and add export files
Other:
- board text added: "Designed By: Kush Nayak AmadorUAVs"
- board text added: "ICP-20100 Breakout Board"
Changed lines of the file:
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@@
       (outputformat 1)
       (mirror false)
-      (drillshape 1)
+      (drillshape 0)
       (scaleselection 1)
-      (outputdirectory "")
+      (outputdirectory "export/")
     )
   )
@@
   )
   (gr_rect (start 100 100) (end 114.5 120.5) (layer "Edge.Cuts") (width 0.2) (fill none))
+  (gr_text "Designed By: Kush Nayak\nAmadorUAVs" (at 112.014 111.76 90) (layer "B.SilkS")
+    (effects (font (size 0.8 0.8) (thickness 0.15)) (justify mirror))
+  )
   (gr_text "SDA" (at 101.1682 112.8014 270) (layer "F.SilkS")
     (effects (font (size 1 0.8) (thickness 0.15)))
@@
     (effects (font (size 1 0.8) (thickness 0.15)))
   )
+  (gr_text "ICP-20100\nBreakout Board" (at 107.188 115.062 270) (layer "F.SilkS")
+    (effects (font (size 0.8 0.8) (thickness 0.15)))
+  )
   (segment (start 108.433408 111.8108) (end 108.926008 111.8108) (width 0.25) (layer "F.Cu") (net 1))
