File: invensense_icm/invensense_icm.kicad_pcb (KiCad board)
At the start: 2 copper layers, 22 x 20.5 mm, 16 parts, among them J1 Conn_01x07, U1 ICM-20608-G, U2 ICM-42688-P, U3 ICM42605

Commit message: Slight modifications to boards and add export files
Parts:
- added C10: 10nF, Capacitor_SMD:C_0603_1608Metric, F.Cu at (112.1, 105.5)
- U3: value ICM42605 -> ICM-42605; footprint Package_LGA:LGA-14_3x2.5mm_P0.5mm_LayoutBorder3x4y -> icm42605-new:PQFN50P300X250X97-14N
- moved R1 1.47 mm to (118.9, 103.4)
- moved C7 1.34 mm to (115.6, 116.4), turned to 90 degrees
- moved C8 1.15 mm to (117.3, 116.4), turned to 90 degrees
- moved R2 1.12 mm to (116.3, 103.4)
- moved R3 0.76 mm to (113.8, 112.9)
- moved C9 0.25 mm to (113.0, 118.8)
Connections:
- C1 pad 1: GND -> +3V3
- C1 pad 2: +3V3 -> GND
- C2 pad 1: GND -> +3V3
- C2 pad 2: +3V3 -> GND
- C7 pad 1: +3V3 -> GND
- C7 pad 2: GND -> +3V3
- C8 pad 1: +3V3 -> GND
- C8 pad 2: GND -> +3V3
- U3 pad 7: unconnected-(U3-Pad7) -> GND
Routing:
- net /SDO: track 42.2 -> 56.8 mm
- net /SDA: track 43.7 -> 56.8 mm
- net +3V3: track 35.1 -> 25.5 mm
- net /SCL: track 47.7 -> 56.7 mm
- net GND: track 17.8 -> 22.7 mm, vias 12 -> 11
- net /~{CS}: track 47.1 -> 44.3 mm, vias 2 -> 3
- net /INT: track 53.9 -> 55.2 mm
Other:
- board text added: "Designed By: Kush Nayak AmadorUAVs"
- board text added: "ICM-Series Breakout Board"
