File: invensense_icm/invensense_icm.kicad_sch (KiCad schematic)
At the start: 16 parts, among them J1 Conn_01x07, U1 ICM-20608-G, U2 ICM-42688-P, U3 ICM42605

Commit message: Slight modifications to boards and add export files
Parts:
- removed U3: ICM42605, Package_LGA:LGA-14_3x2.5mm_P0.5mm_LayoutBorder3x4y, symbol ICM-42605:ICM42605
- added C10: 10nF, Capacitor_SMD:C_0603_1608Metric, symbol Device:C
- added U3: ICM-42605, icm42605-new:PQFN50P300X250X97-14N, symbol icm42605-new:ICM-42605
Connections:
- net +3V3: now also C1.1, C2.1, C7.2, C8.2, C10.1, U3.5 (VDDIO), U3.8 (VDD); no longer C1.2, C2.2, C7.1, C8.1
- net GND: now also C1.2, C2.2, C7.1, C8.1, C10.2, U3.6 (GND), U3.7 (RESV_3), U3.9 (INT2/FSYNC); no longer C1.1, C2.1, C7.2, C8.2
- net INT: now also U3.4 (INT1/INT)
- net SCL: now also J1.3 (Pin_3), U3.13 (AP_SCL/AP_SCLK); no longer J1.4 (Pin_4)
- net SDA: now also J1.4 (Pin_4), U3.14 (AP_SDA/AP_SDIO/AP_SDI); no longer J1.5 (Pin_5)
- net SDO: now also J1.5 (Pin_5), U3.1 (AP_SDO/AP_ADO); no longer J1.6 (Pin_6)
- net ~{CS}: now also J1.6 (Pin_6), U3.12 (AP_CS); no longer J1.3 (Pin_3)
- no-connect marks 4 -> 8
Other:
- moved on the sheet: C1, C2, C7, C8, C9, J1, R3
